File: CMS32L032GE24SS-SoM/PowerRegulator.kicad_sch (KiCad schematic)
At the start: 6 parts, among them U301 AP2127K-ADJ

Commit message: updated Part number in LCSC
Parts:
- C301, C302: LCSC (none) -> C116352; Vendor (none) -> SAMSUNG(三星); Vendor Model (none) -> CL21B105KAFNNNE
- C303: LCSC (none) -> C107151; Vendor (none) -> YAGEO(国巨); Vendor Model (none) -> CC0805KRX7R9BB391
- R301: LCSC (none) -> C483186; Vendor (none) -> YAGEO(国巨); Vendor Model (none) -> RC0805FR-0756K2L
- R302: LCSC (none) -> C17506; Vendor (none) -> UNI-ROYAL(厚声); Vendor Model (none) -> 0805W8F1802T5E
- U301: LCSC (none) -> C96343; Vendor (none) -> DIODES(美台); Vendor Model (none) -> AP2127K-ADJTRG1
Changed lines of the file:
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@@
       (effects (font (size 1.27 1.27)) hide)
     )
-    (property "Description" "" (at 93.98 95.885 0)
+    (property "Description" "电阻类型: 厚膜电阻 阻值: 56.2kΩ 精度: ±1% 功率: 125mW 温度系数: ±100ppm/℃ 最大工作电压: 150V 工作温度范围: -55℃~+155℃" (at 93.98 95.885 0)
       (effects (font (size 1.27 1.27)) hide)
     )
-    (property "LCSC" "" (at 93.98 95.885 0)
+    (property "LCSC" "C483186" (at 93.98 95.885 0)
       (effects (font (size 1.27 1.27)) hide)
     )
-    (property "Vendor" "" (at 93.98 95.885 0)
+    (property "Vendor" "YAGEO(国巨)" (at 93.98 95.885 0)
       (effects (font (size 1.27 1.27)) hide)
     )
-    (property "Vendor Model" "" (at 93.98 95.885 0)
+    (property "Vendor Model" "RC0805FR-0756K2L" (at 93.98 95.885 0)
       (effects (font (size 1.27 1.27)) hide)
     )
@@
       (effects (font (size 1.27 1.27)) hide)
     )
-    (property "Description" "" (at 55.88 100.33 0)
+    (property "Description" "容值: 1uF 精度: ±10% 额定电压: 25V 材质(温度系数): X7R 材质：X7R" (at 55.88 100.33 0)
       (effects (font (size 1.27 1.27)) hide)
     )
-    (property "LCSC" "" (at 55.88 100.33 0)
+    (property "LCSC" "C116352" (at 55.88 100.33 0)
       (effects (font (size 1.27 1.27)) hide)
     )
-    (property "Vendor" "" (at 55.88 100.33 0)
+    (property "Vendor" "SAMSUNG(三星)" (at 55.88 100.33 0)
       (effects (font (size 1.27 1.27)) hide)
     )
-    (property "Vendor Model" "" (at 55.88 100.33 0)
+    (property "Vendor Model" "CL21B105KAFNNNE" (at 55.88 100.33 0)
       (effects (font (size 1.27 1.27)) hide)
     )
@@
       (effects (font (size 1.27 1.27)) hide)
     )
-    (property "Description" "" (at 106.68 100.965 0)
+    (property "Description" "容值: 1uF 精度: ±10% 额定电压: 25V 材质(温度系数): X7R 材质：X7R" (at 106.68 100.965 0)
       (effects (font (size 1.27 1.27)) hide)
     )
-    (property "LCSC" "" (at 106.68 100.965 0)
+    (property "LCSC" "C116352" (at 106.68 100.965 0)
       (effects (font (size 1.27 1.27)) hide)
     )
-    (property "Vendor" "" (at 106.68 100.965 0)
+    (property "Vendor" "SAMSUNG(三星)" (at 106.68 100.965 0)
       (effects (font (size 1.27 1.27)) hide)
     )
-    (property "Vendor Model" "" (at 106.68 100.965 0)
+    (property "Vendor Model" "CL21B105KAFNNNE" (at 106.68 100.965 0)
       (effects (font (size 1.27 1.27)) hide)
     )
@@
       (effects (font (size 1.27 1.27)) hide)
     )
-    (property "Description" "" (at 99.06 106.045 0)
+    (property "Description" "容值: 390pF 精度: ±10% 额定电压: 50V 材质(温度系数): X7R 材质：X7R" (at 99.06 106.045 0)
       (effects (font (size 1.27 1.27)) hide)
     )
-    (property "LCSC" "" (at 99.06 106.045 0)
+    (property "LCSC" "C107151" (at 99.06 106.045 0)
       (effects (font (size 1.27 1.27)) hide)
     )
-    (property "Vendor" "" (at 99.06 106.045 0)
+    (property "Vendor" "YAGEO(国巨)" (at 99.06 106.045 0)
       (effects (font (size 1.27 1.27)) hide)
     )
-    (property "Vendor Model" "" (at 99.06 106.045 0)
+    (property "Vendor Model" "CC0805KRX7R9BB391" (at 99.06 106.045 0)
       (effects (font (size 1.27 1.27)) hide)
     )
@@
       (effects (font (size 1.27 1.27)) hide)
     )
-    (property "Description" "" (at 88.265 106.045 0)
+    (property "Description" "电阻类型: 厚膜电阻 阻值: 18kΩ 精度: ±1% 功率: 125mW 温度系数: ±100ppm/℃ 最大工作电压: 150V 工作温度范围: -55℃~+155℃" (at 88.265 106.045 0)
       (effects (font (size 1.27 1.27)) hide)
     )
-    (property "LCSC" "" (at 88.265 106.045 0)
+    (property "LCSC" "C17506" (at 88.265 106.045 0)
       (effects (font (size 1.27 1.27)) hide)
     )
-    (property "Vendor" "" (at 88.265 106.045 0)
+    (property "Vendor" "UNI-ROYAL(厚声)" (at 88.265 106.045 0)
       (effects (font (size 1.27 1.27)) hide)
     )
-    (property "Vendor Model" "" (at 88.265 106.045 0)
+    (property "Vendor Model" "0805W8F1802T5E" (at 88.265 106.045 0)
       (effects (font (size 1.27 1.27)) hide)
     )
@@
       (effects (font (size 1.27 1.27)) hide)
     )
-    (property "Description" "" (at 78.74 95.885 0)
+    (property "Description" "输出类型: 可调 输出极性: 正 输出通道数: 1 最大输入电压: 6V 输出电压: 0.8V~5.5V 压差: 300mV@(300mA) 静态" (at 78.74 95.885 0)
       (effects (font (size 1.27 1.27)) hide)
     )
-    (property "LCSC" "" (at 78.74 95.885 0)
+    (property "LCSC" "C96343" (at 78.74 95.885 0)
       (effects (font (size 1.27 1.27)) hide)
     )
-    (property "Vendor" "" (at 78.74 95.885 0)
+    (property "Vendor" "DIODES(美台)" (at 78.74 95.885 0)
       (effects (font (size 1.27 1.27)) hide)
     )
-    (property "Vendor Model" "" (at 78.74 95.885 0)
+    (property "Vendor Model" "AP2127K-ADJTRG1" (at 78.74 95.885 0)
       (effects (font (size 1.27 1.27)) hide)
     )
