File: CMS32L051LQ48-nano/CMS32L051LQ48-nano.kicad_sch (KiCad schematic)
At the start: 9 parts, among them J103 USB_B_Micro, J105 Connection to DAPLink Board

Commit message: Changed USB micro B connector
Parts:
- J103: footprint Connector_USB:USB_Micro-B_GCT_USB3076-30-A -> Connector_USB:USB_Micro-B_XKB_U254-051T-4BH83-F1S; LCSC (none) -> C397452; Vendor (none) -> XKB Connectivity(中国星坤); Vendor Model (none) -> U254-051T-4BH83-F1S
Changed lines of the file:
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@@
       (effects (font (size 1.27 1.27)))
     )
-    (property "Footprint" "Connector_USB:USB_Micro-B_GCT_USB3076-30-A" (at 48.26 83.82 0)
+    (property "Footprint" "Connector_USB:USB_Micro-B_XKB_U254-051T-4BH83-F1S" (at 48.26 83.82 0)
       (effects (font (size 1.27 1.27)) hide)
     )
@@
       (effects (font (size 1.27 1.27)) hide)
     )
+    (property "Description" "连接器类型: Micro-B 标准: USB 2.0 公母: 母座 触点数量: 5 端口数量: 1 安装方式: 卧贴 额定电流 - 电源: 1.8A 触" (at 44.45 82.55 0)
+      (effects (font (size 1.27 1.27)) hide)
+    )
+    (property "LCSC" "C397452" (at 44.45 82.55 0)
+      (effects (font (size 1.27 1.27)) hide)
+    )
+    (property "Vendor" "XKB Connectivity(中国星坤)" (at 44.45 82.55 0)
+      (effects (font (size 1.27 1.27)) hide)
+    )
+    (property "Vendor Model" "U254-051T-4BH83-F1S" (at 44.45 82.55 0)
+      (effects (font (size 1.27 1.27)) hide)
+    )
