File: DisplayConverterTesterBoard/JDI_MemoryLCD_0.96in.kicad_sch (KiCad schematic)
At the start: 0 parts

Commit message: added connector for 0.96in
Parts:
- added C?: 0.1u 10V, symbol Device:C
- added C?: 1u 10V, symbol Device:C
- added J?: BM20B(0.8)-10DS-0.4V, symbol Connector_Generic_MountingPin:Conn_02x05_Counter_Clockwise_MountingPin
Connections:
- new net 3V3: C?.1, J?.9 (Pin_9)
- new net DISP: C?.1, J?.2 (Pin_2)
- new net GND: C?.2, C?.2, J?.1 (Pin_1), J?.10 (Pin_10), J?.MP (MountPin)
- new net MOSI: J?.7 (Pin_7)
- new net SCK: J?.4 (Pin_4)
- new net ~{SCS}: J?.3 (Pin_3)
- no-connect marks 0 -> 3

Commit message: annotate all components
Parts:
- gave numbers to parts that had none: 1
Changed lines of the file:
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@@
         )
         (path "/58d9d6aa-d5e3-4b7b-b546-d57c329de758/edcee65f-25a8-4aef-871d-10e28d870fa2"
-          (reference "C?") (unit 1)
+          (reference "C9") (unit 1)
         )
       )
@@
         )
         (path "/58d9d6aa-d5e3-4b7b-b546-d57c329de758/edcee65f-25a8-4aef-871d-10e28d870fa2"
-          (reference "C?") (unit 1)
+          (reference "C8") (unit 1)
         )
       )
@@
   (symbol (lib_id "Connector_Generic_MountingPin:Conn_02x05_Counter_Clockwise_MountingPin") (at 137.16 63.5 0) (unit 1)
     (in_bom yes) (on_board yes) (dnp no) (fields_autoplaced)
-    (property "Reference" "J?" (at 138.43 52.07 0)
+    (property "Reference" "J5" (at 138.43 52.07 0)
       (effects (font (size 1.27 1.27)))
     )
@@
       (project "DisplayConverterTesterBoard"
         (path "/58d9d6aa-d5e3-4b7b-b546-d57c329de758/edcee65f-25a8-4aef-871d-10e28d870fa2"
-          (reference "J?") (unit 1)
+          (reference "J5") (unit 1)
         )
       )

Commit message: set components LCSC
Parts:
- C?: footprint (none) -> Capacitor_SMD:C_0805_2012Metric_Pad1.18x1.45mm_HandSolder; LCSC (none) -> C1853551; Vendor (none) -> YAGEO(国巨); Vendor Model (none) -> CC0805JKX7R0BB104
- C?: footprint (none) -> Resistor_SMD:R_0805_2012Metric_Pad1.20x1.40mm_HandSolder; LCSC (none) -> C28323; Vendor (none) -> SAMSUNG(三星); Vendor Model (none) -> CL21B105KBFNNNE
- J5: LCSC (none) -> C424532; Vendor (none) -> HRS(广濑); Vendor Model (none) -> BM20B(0.8)-10DS-0.4V(
Changed lines of the file:
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@@
       (effects (font (size 1.27 1.27)) (justify left))
     )
-    (property "Footprint" "" (at 101.2952 100.33 0)
+    (property "Footprint" "Capacitor_SMD:C_0805_2012Metric_Pad1.18x1.45mm_HandSolder" (at 101.2952 100.33 0)
       (effects (font (size 1.27 1.27)) hide)
     )
     (property "Datasheet" "~" (at 100.33 96.52 0)
+      (effects (font (size 1.27 1.27)) hide)
+    )
+    (property "Description" "容值: 100nF 精度: ±5% 额定电压: 100V 材质(温度系数): X7R " (at 100.33 96.52 0)
+      (effects (font (size 1.27 1.27)) hide)
+    )
+    (property "LCSC" "C1853551" (at 100.33 96.52 0)
+      (effects (font (size 1.27 1.27)) hide)
+    )
+    (property "Vendor" "YAGEO(国巨)" (at 100.33 96.52 0)
+      (effects (font (size 1.27 1.27)) hide)
+    )
+    (property "Vendor Model" "CC0805JKX7R0BB104" (at 100.33 96.52 0)
       (effects (font (size 1.27 1.27)) hide)
     )
@@
       (effects (font (size 1.27 1.27)) (justify left))
     )
-    (property "Footprint" "" (at 82.8548 100.33 0)
+    (property "Footprint" "Resistor_SMD:R_0805_2012Metric_Pad1.20x1.40mm_HandSolder" (at 82.8548 100.33 0)
       (effects (font (size 1.27 1.27)) hide)
     )
     (property "Datasheet" "~" (at 83.82 96.52 0)
+      (effects (font (size 1.27 1.27)) hide)
+    )
+    (property "Description" "容值: 1uF 精度: ±10% 额定电压: 50V 材质(温度系数): X7R 材质:X7R" (at 83.82 96.52 0)
+      (effects (font (size 1.27 1.27)) hide)
+    )
+    (property "LCSC" "C28323" (at 83.82 96.52 0)
+      (effects (font (size 1.27 1.27)) hide)
+    )
+    (property "Vendor" "SAMSUNG(三星)" (at 83.82 96.52 0)
+      (effects (font (size 1.27 1.27)) hide)
+    )
+    (property "Vendor Model" "CL21B105KBFNNNE" (at 83.82 96.52 0)
       (effects (font (size 1.27 1.27)) hide)
     )
@@
       (effects (font (size 1.27 1.27)) hide)
     )
+    (property "Description" "间距: 0.4mm PIN总数: 10 行数: 2 公母: 母 安装方式: 立贴 额定电流: 300mA 触头镀层: 金 工作温度范围: " (at 137.16 63.5 0)
+      (effects (font (size 1.27 1.27)) hide)
+    )
+    (property "LCSC" "C424532" (at 137.16 63.5 0)
+      (effects (font (size 1.27 1.27)) hide)
+    )
+    (property "Vendor" "HRS(广濑)" (at 137.16 63.5 0)
+      (effects (font (size 1.27 1.27)) hide)
+    )
+    (property "Vendor Model" "BM20B(0.8)-10DS-0.4V(" (at 137.16 63.5 0)
+      (effects (font (size 1.27 1.27)) hide)
+    )

Commit message: added datasheet for BM20
Parts:
- J5: Vendor Model BM20B(0.8)-10DS-0.4V( -> BM20B(0.8)-10DS-0.4V
Changed lines of the file:
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@@
       (effects (font (size 1.27 1.27)) hide)
     )
-    (property "Datasheet" "~" (at 137.16 63.5 0)
+    (property "Datasheet" "https://www.hirose.com/en/product/document?clcode=CL0684-9008-4-51&productname=BM20B(0.8)-10DS-0.4V(51)&series=BM20&documenttype=Catalog&lang=en&documentid=D47513_en" (at 137.16 63.5 0)
       (effects (font (size 1.27 1.27)) hide)
     )
@@
       (effects (font (size 1.27 1.27)) hide)
     )
-    (property "Vendor Model" "BM20B(0.8)-10DS-0.4V(" (at 137.16 63.5 0)
+    (property "Vendor Model" "BM20B(0.8)-10DS-0.4V" (at 137.16 63.5 0)
       (effects (font (size 1.27 1.27)) hide)
     )

Commit message: added hirose BM20 connectors
Parts:
- J5: footprint (none) -> IotPi_Connector_Hirose:BM20B(0.8)-10DS-0.4V
Changed lines of the file:
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@@
     (stroke (width 0) (type default))
   )
-  (wire (pts (xy 152.4 58.42) (xy 144.78 58.42))
+  (wire (pts (xy 144.78 58.42) (xy 152.4 58.42))
     (stroke (width 0) (type default))
   )
@@
     (stroke (width 0) (type default))
   )
-  (wire (pts (xy 152.4 60.96) (xy 144.78 60.96))
-    (stroke (width 0) (type default))
-  )
-  (wire (pts (xy 152.4 66.04) (xy 144.78 66.04))
+  (wire (pts (xy 144.78 60.96) (xy 152.4 60.96))
+    (stroke (width 0) (type default))
+  )
+  (wire (pts (xy 144.78 66.04) (xy 152.4 66.04))
     (stroke (width 0) (type default))
   )
@@
   )
   (symbol (lib_id "Connector_Generic_MountingPin:Conn_02x05_Counter_Clockwise_MountingPin") (at 137.16 63.5 0) (unit 1)
-    (in_bom yes) (on_board yes) (dnp no) (fields_autoplaced)
+    (in_bom yes) (on_board yes) (dnp no)
     (property "Reference" "J5" (at 138.43 52.07 0)
       (effects (font (size 1.27 1.27)))
@@
       (effects (font (size 1.27 1.27)))
     )
-    (property "Footprint" "" (at 137.16 63.5 0)
-      (effects (font (size 1.27 1.27)) hide)
-    )
+    (property "Footprint" "IotPi_Connector_Hirose:BM20B(0.8)-10DS-0.4V" (at 137.16 63.5 0)
+      (effects (font (size 1.27 1.27)) hide)
+    )
