File: DisplayConverterTesterBoard/DisplayConverterTesterBoard.kicad_pcb (KiCad board)
At the start: 2 copper layers, 37 x 36 mm, 25 parts, among them J2 Conn_01x07, J3 Conn_01x03, J4 FPC 20PIN P0.5mm, J5 BM20B(0.8)-10DS-0.4V, J6 Conn_01x03, J7 FPC 10PIN P0.5mm, U2 TPS61040DBV

Commit message: added more Texts
Other:
- board text added: "VDD"
- board text added: "VSS"
Changed lines of the file:
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@@
+    (effects (font (size 1 1) (thickness 0.15)) (justify left bottom))
+  )
+  (gr_text "EXT MODE" (at 99.568 82.55) (layer "F.SilkS")
     (effects (font (size 1 1) (thickness 0.15)) (justify left bottom))
   )
@@
     (effects (font (size 1 1) (thickness 0.15)) (justify left bottom))
   )
+  (gr_text "VDD" (at 104.267 85.344) (layer "F.SilkS")
+    (effects (font (size 1 1) (thickness 0.15)) (justify left bottom))
+  )
+  (gr_text "VSS" (at 104.521 79.883) (layer "F.SilkS")
+    (effects (font (size 1 1) (thickness 0.15)) (justify left bottom))
+  )

Commit message: added more Texts
Other:
- board text added: "JDI 0.96{dblquote}"
- board text added: "JDI 1.28{dblquote}"
- board text added: "OLED 0.6{dblquote}"
Changed lines of the file:
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@@
+    (effects (font (size 1 1) (thickness 0.15)) (justify left bottom))
+  )
+  (gr_text "JDI 1.28{dblquote}" (at 115.062 78.74) (layer "F.SilkS")
     (effects (font (size 1 1) (thickness 0.15)) (justify left bottom))
   )
@@
     (effects (font (size 1 1) (thickness 0.15)) (justify left bottom))
   )
+  (gr_text "JDI 0.96{dblquote}" (at 99.314 94.615) (layer "F.SilkS")
+    (effects (font (size 1 1) (thickness 0.15)) (justify left bottom))
+  )
   (gr_text "VDD" (at 104.267 85.344) (layer "F.SilkS")
     (effects (font (size 1 1) (thickness 0.15)) (justify left bottom))
   )
+  (gr_text "OLED 0.6{dblquote}" (at 122.301 72.771 90) (layer "F.SilkS")
+    (effects (font (size 1 1) (thickness 0.15)) (justify left bottom))
+  )
